Commit message: reinitilzed local git repo after mistakenly add local repo to root ws directory. Finished Task 1 & 2 of checkpoint

File: rb1_ros2_description/urdf/elevator/elevator.urdf.xacro (robot description, xacro)
@@ -60,5 +60,5 @@
 			<child link="${prefix}_platform_link" />
 			<axis xyz="0 0 1"/>
-			<limit effort="10.0" lower="0.0" upper="0.034" velocity="0.5"/>
+			<limit effort="10.0" lower="-0.01" upper="0.034" velocity="0.5"/>
 	</joint>
 	<link name="${prefix}_platform_link">

File: rb1_ros2_description/xacro/rb1_ros2_base.urdf.xacro (robot description, xacro)
@@ -18,4 +18,6 @@
 	<!-- Import Elevator -->
 	<xacro:include filename="$(find rb1_ros2_description)/urdf/elevator/elevator.urdf.xacro"/>
+    <!-- Import ros2_control framework -->
+    <xacro:include filename="$(find rb1_ros2_description)/xacro/ros2_control.urdf.xacro"/>
 	<!-- ***************** -->
 	<!-- Global parameters -->
@@ -79,4 +81,4 @@
 	</xacro:sensor_hokuyo_ust20lx>
 	<!-- Gazebo ros2 control plugins -->
-	<!-- <xacro:ros2_control/> -->
+	<xacro:ros2_control name="rb1_ros2_control" prefix="$(arg prefix)"/>
 </robot>
